File: FluidNC-PCB/FluidNC-PCB.kicad_pcb (KiCad board)
At the start: 2 copper layers, 54 parts, among them J1 Conn_01x04_Pin, J11 Molex_01x02_Socket, J12 Molex_01x02_Socket, J13 Molex_01x02_Socket, J14 Molex_01x02_Socket, J15 Molex_01x02_Socket, J16 Molex_01x02_Socket, J17 Molex_01x02_Socket, J18 Molex_01x02_Socket, J19 Molex_01x02_Socket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

Commit message: Finished (version 1) of PCB
Parts:
- removed H5, H6: MountingHole, MountingHole:MountingHole_3.2mm_M3
- removed J19: Molex_01x02_Socket, Connector_Molex:Molex_KK-254_AE-6410-02A_1x02_P2.54mm_Vertical
- moved H2 170.7 mm to (81.5, 141.5)
- moved J8 74.8 mm to (198.2, 128.5), turned to 90 degrees
- moved H4 63.9 mm to (204.5, 141.5)
- moved H3 62.9 mm to (204.5, 59.0)
- moved J16 58.8 mm to (177.5, 105.0), turned to 90 degrees
- moved J7 57.5 mm to (198.0, 115.0), turned to 90 degrees
- moved J13 53.8 mm to (177.5, 131.0), turned to 90 degrees
- moved R9 51.1 mm to (162.7, 103.5)
- moved J15 49.7 mm to (177.5, 111.5), turned to 90 degrees
- moved R8 46.8 mm to (162.7, 108.5)
- moved J12 46.0 mm to (177.5, 124.5), turned to 90 degrees
- moved R1 45.8 mm to (167.3, 113.5), turned to 180 degrees
- moved J17 42.7 mm to (187.0, 105.5)
- moved J14 39.5 mm to (177.5, 137.5), turned to 90 degrees
- moved J11 39.1 mm to (177.5, 118.0), turned to 90 degrees
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Connections:
- U2 pad 10: M2_DIR -> M1_DIR
- U2 pad 11: M2_STP -> M1_STP
- U2 pad 12: M3_DIR -> M2_DIR
- U2 pad 13: M3_STP -> M2_STP
- U2 pad 23: Net-(J19-Pin_2) -> unconnected-(U2-D5-Pad23)
- U2 pad 24: Net-(J19-Pin_1) -> unconnected-(U2-D18-Pad24)
- U2 pad 25: M5_STP -> M5_DIR
- U2 pad 26: M5_DIR -> M5_STP
- U2 pad 29: M4_STP -> M4_DIR
- U2 pad 30: M4_DIR -> M4_STP
- U2 pad 6: M0_DIR -> M3_DIR
- U2 pad 7: M0_STP -> M3_STP
- U2 pad 8: M1_DIR -> M0_DIR
- U2 pad 9: M1_STP -> M0_STP
Routing:
- net +3.3V: track 202.5 -> 594.9 mm
- net ENABLE_N: track 91.2 -> 293.0 mm
- net +12V: track 249.4 -> 380.7 mm
- net Net-(J11-Pin_2): track 0.00 -> 104.6 mm
- net Net-(A1-MS3): track 88.5 -> 193.0 mm
- net Net-(A1-MS2): track 88.7 -> 192.4 mm
- net Net-(J12-Pin_2): track 0.00 -> 101.7 mm
- net Net-(A1-MS1): track 95.5 -> 196.6 mm
- net Net-(J13-Pin_2): track 0.00 -> 96.8 mm
- net Net-(J14-Pin_2): track 0.00 -> 91.9 mm
- net M5_DIR: track 0.00 -> 60.7 mm
- net M5_STP: track 0.00 -> 57.1 mm
- net Net-(J16-Pin_2): track 0.00 -> 53.8 mm
- net M3_STP: track 0.00 -> 50.6 mm
- net Net-(J15-Pin_2): track 0.00 -> 50.5 mm
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- added copper zone on F.Cu, net GND
- removed copper zone on B.Cu, net GND
Other:
- board outline added: 133 x 92.5 mm
